File: esp32s3_adc_mini_bat/BAT.kicad_sch (KiCad schematic)
At the start: 10 parts, among them CN2 B2B-PH-K-S, SW3 XDMK-12C01-25, U4 TP4056_C382139

Commit message: chore: silk screen cleanup and DRC pass
Parts:
- R10: value 560 -> 330
Changed lines of the file:
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@@
 			)
 		)
-		(property "Value" "560"
+		(property "Value" "330"
 			(at 165.1 114.2999 0)
 			(show_name no)
