File: esp32s3_adc_mini_bat/ESP32S3WROOM1.kicad_sch (KiCad schematic)
At the start: 5 parts, among them J4 Conn_01x22_Socket, J5 Conn_01x22_Socket, U2 ESP32-S3-WROOM-1

Commit message: chore: silk screen cleanup and DRC pass
Parts:
- J4, J5: now not fitted; now left out of the parts list
Changed lines of the file:
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@@
 		(body_style 1)
 		(exclude_from_sim no)
-		(in_bom yes)
-		(on_board yes)
-		(in_pos_files yes)
-		(dnp no)
+		(in_bom no)
+		(on_board yes)
+		(in_pos_files no)
+		(dnp yes)
 		(property "Reference" "J5"
 			(at 243.078 107.95 90)
@@
 		(body_style 1)
 		(exclude_from_sim no)
-		(in_bom yes)
-		(on_board yes)
-		(in_pos_files yes)
-		(dnp no)
+		(in_bom no)
+		(on_board yes)
+		(in_pos_files no)
+		(dnp yes)
 		(property "Reference" "J4"
 			(at 178.308 117.348 90)
