File: esp32s3_adc_mini_bat/esp32s3_adc_mini_bat.kicad_pcb (KiCad board)
At the start: 2 copper layers, 42 x 61 mm, 59 parts, among them CN1 PJ-320D, CN2 B2B-PH-K-S, J1 USB_C_Receptacle_USB2.0_16P, J4 Conn_01x22_Socket, J5 Conn_01x22_Socket, SW1 TS-1088-AR02016, SW2 TS-1088-AR02016, SW3 XDMK-12C01-25, U1 USBLC6-2SC6, U2 ESP32-S3-WROOM-1, U3 AP2112K-3.3, U4 TP4056_C382139, U5 ES8388

Commit message: chore: silk screen cleanup and DRC pass
Parts:
- removed R3: 0R, Resistor_SMD:R_0402_1005Metric
- R10: value 560 -> 330
- moved R9 11.2 mm to (147.4, 99.1)
- moved D4 10.7 mm to (148.2, 97.8)
- moved D5 10.7 mm to (148.2, 96.5)
- moved U4 10.7 mm to (153.3, 97.2)
- moved R10 9.94 mm to (147.3, 95.3)
- moved R8 7.92 mm to (156.2, 100.5), turned to 0 degrees
- moved C2 5.05 mm to (139.4, 103.0)
- moved C1 5.05 mm to (143.7, 103.2)
- moved C23 4.74 mm to (159.8, 99.7)
- moved R14 4.54 mm to (153.4, 82.5), turned to -90 degrees
- moved CN1 4.00 mm to (160.0, 106.6)
- moved D1 4.00 mm to (143.8, 105.2)
- moved H3 4.00 mm to (168.5, 108.5)
- moved H4 4.00 mm to (137.5, 108.5)
- moved J1 4.00 mm to (148.2, 111.2)
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- renumbered CN2 to BAT, SW2 to BOT, SW3 to PWR, SW1 to RST
Connections:
- C1 pad 1: Net-(D1-K) -> VBUS
- D1 pad 1: Net-(D1-K) -> VBUS
- J1 pad A4: Net-(D1-K) -> VBUS
- J1 pad A9: Net-(D1-K) -> VBUS
- J1 pad B4: Net-(D1-K) -> VBUS
- J1 pad B9: Net-(D1-K) -> VBUS
- U5 pad 18: /CODEC/CODEC_AGND -> GND
- U5 pad 29: /CODEC/CODEC_AGND -> GND
Routing:
- net +3V3: track 36.9 -> 122.0 mm, vias 1 -> 3
- net VBUS: track 0.00 -> 58.9 mm, vias 0 -> 1
- net I2C_CLK: track 0.00 -> 23.5 mm, vias 0 -> 2
- net I2C_DAT: track 11.8 -> 33.2 mm, vias 0 -> 2
- net Net-(D3-A): track 0.00 -> 19.6 mm
- net BCK: track 13.6 -> 30.6 mm, vias 0 -> 2
- net Net-(U5-RIN1): track 0.00 -> 16.0 mm, vias 0 -> 2
- net Net-(U5-LIN1): track 0.00 -> 15.9 mm
- net LDO_IN: track 4.49 -> 16.9 mm, vias 2 -> 0
- net Net-(D1-K): track 9.88 -> 0.00 mm
- net SCKI: track 30.0 -> 38.7 mm, vias 0 -> 1
- net Net-(CN2-Pad2): track 0.00 -> 8.49 mm
- net LRCK: track 16.9 -> 23.8 mm, vias 0 -> 2
- net GND: track 0.00 -> 6.55 mm, vias 5 -> 23
- net LINE-IN-L: track 0.00 -> 4.61 mm
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Other:
- board size 42 x 61 mm -> 42 x 57 mm
- board text added: "NOP"

Commit message: chore: minor changes
Routing:
- net GND: vias 23 -> 41
Changed lines of the file:
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@@
 			(at 1.635 -0.04 0)
 			(layer "F.SilkS")
+			(hide yes)
 			(effects
 				(font
@@
 			(at 1.625 0.01 180)
 			(layer "F.SilkS")
+			(hide yes)
 			(effects
 				(font
@@
 		)
 	)
+	(dimension
+		(type orthogonal)
+		(layer "F.SilkS")
+		(pts
+			(xy 132 57) (xy 132 114)
+		)
+		(height -7.5)
+		(orientation 1)
+		(format
+			(prefix "")
+			(suffix "")
+			(units 3)
+			(units_format 0)
+			(precision 4)
+			(suppress_zeroes yes)
+		)
+		(style
+			(thickness 0.1)
+			(arrow_length 1.27)
+			(text_position_mode 0)
+			(arrow_direction outward)
+			(extension_height 0.58642)
+			(extension_offset 0.5)
+			(keep_text_aligned yes)
+		)
+		(gr_text "57"
+			(at 123.4 85.5 90)
+			(layer "F.SilkS")
+			(effects
+				(font
+					(size 1 1)
+					(thickness 0.1)
+				)
+			)
+		)
+	)
+	(dimension
+		(type orthogonal)
+		(layer "F.SilkS")
+		(pts
+			(xy 174 113.9925) (xy 132 114)
+		)
+		(height 8.5075)
+		(orientation 0)
+		(format
+			(prefix "")
+			(suffix "")
+			(units 3)
+			(units_format 0)
+			(precision 4)
+			(suppress_zeroes yes)
+		)
+		(style
+			(thickness 0.1)
+			(arrow_length 1.27)
+			(text_position_mode 0)
+			(arrow_direction outward)
+			(extension_height 0.58642)
+			(extension_offset 0.5)
+			(keep_text_aligned yes)
+		)
+		(gr_text "42"
+			(at 153 121.4 0)
+			(layer "F.SilkS")
+			(effects
+				(font
+					(size 1 1)
+					(thickness 0.1)
+				)
+			)
+		)
+	)
 	(segment
 		(start 140.42 93.32)
@@
 	)
 	(via
+		(at 151.5 101.5)
+		(size 0.6)
+		(drill 0.3)
+		(layers "F.Cu" "B.Cu")
+		(free yes)
+		(net "GND")
+	)
+	(via
 		(at 156.24875 87.9725)
 		(size 0.6)
@@
 	)
 	(via
+		(at 156.5 71.5)
+		(size 0.6)
+		(drill 0.3)
+		(layers "F.Cu" "B.Cu")
+		(free yes)
+		(net "GND")
+	)
+	(via
 		(at 144.945 88.354)
 		(size 0.6)
@@
 	)
 	(via
+		(at 141.5 105)
+		(size 0.6)
+		(drill 0.3)
+		(layers "F.Cu" "B.Cu")
+		(free yes)
+		(net "GND")
+	)
+	(via
+		(at 169 101.5)
+		(size 0.6)
+		(drill 0.3)
+		(layers "F.Cu" "B.Cu")
+		(free yes)
+		(net "GND")
+	)
+	(via
 		(at 151.45 107.43)
 		(size 0.6)
@@
 	)
 	(via
+		(at 143.5 90.5)
+		(size 0.6)
+		(drill 0.3)
+		(layers "F.Cu" "B.Cu")
+		(free yes)
+		(net "GND")
+	)
+	(via
+		(at 148.5 60.5)
+		(size 0.6)
+		(drill 0.3)
+		(layers "F.Cu" "B.Cu")
+		(free yes)
+		(net "GND")
+	)
+	(via
+		(at 169.5 95.5)
+		(size 0.6)
+		(drill 0.3)
+		(layers "F.Cu" "B.Cu")
+		(free yes)
+		(net "GND")
+	)
+	(via
 		(at 156.24875 85.1975)
 		(size 0.6)
@@
 	)
 	(via
+		(at 163 85.5)
+		(size 0.6)
+		(drill 0.3)
+		(layers "F.Cu" "B.Cu")
+		(free yes)
+		(net "GND")
+	)
+	(via
+		(at 150.88875 86.6)
+		(size 0.6)
+		(drill 0.3)
+		(layers "F.Cu" "B.Cu")
+		(net "GND")
+	)
+	(via
+		(at 156.5 64)
+		(size 0.6)
+		(drill 0.3)
+		(layers "F.Cu" "B.Cu")
+		(free yes)
+		(net "GND")
+	)
+	(via
 		(at 145.61 84.04)
 		(size 0.6)
@@
 	)
 	(via
+		(at 164.5 105)
+		(size 0.6)
+		(drill 0.3)
+		(layers "F.Cu" "B.Cu")
+		(free yes)
+		(net "GND")
+	)
+	(via
+		(at 156.5 60.5)
+		(size 0.6)
+		(drill 0.3)
+		(layers "F.Cu" "B.Cu")
+		(free yes)
+		(net "GND")
+	)
+	(via
+		(at 159.5 93)
+		(size 0.6)
+		(drill 0.3)
+		(layers "F.Cu" "B.Cu")
+		(free yes)
+		(net "GND")
+	)
+	(via
 		(at 154.44 85.18)
 		(size 0.6)
@@
 	)
 	(via
+		(at 145.5 101.5)
+		(size 0.6)
+		(drill 0.3)
+		(layers "F.Cu" "B.Cu")
+		(free yes)
+		(net "GND")
+	)
+	(via
+		(at 158.5 82.5)
+		(size 0.6)
+		(drill 0.3)
+		(layers "F.Cu" "B.Cu")
+		(free yes)
+		(net "GND")
+	)
+	(via
 		(at 145.44 81.02)
 		(size 0.6)
@@
 	)
 	(via
-		(at 150.88875 86.6)
+		(at 169.5 97)
 		(size 0.6)
 		(drill 0.3)
 		(layers "F.Cu" "B.Cu")
+		(free yes)
 		(net "GND")
 	)
@@
 	)
 	(via
+		(at 156.5 67.5)
+		(size 0.6)
+		(drill 0.3)
+		(layers "F.Cu" "B.Cu")
+		(free yes)
+		(net "GND")
+	)
+	(via
+		(at 142.5 84.5)
+		(size 0.6)
+		(drill 0.3)
+		(layers "F.Cu" "B.Cu")
+		(free yes)
+		(net "GND")
+	)
+	(via
 		(at 145.05 107.43)
 		(size 0.6)
@@
 		(net "GND")
 	)
+	(via
+		(at 152.5 60.5)
+		(size 0.6)
+		(drill 0.3)
+		(layers "F.Cu" "B.Cu")
+		(free yes)
+		(net "GND")
+	)
